File: hardware/main_board/motor_drivers.sch (KiCad schematic (older format))
At the start: 6 parts, among them J301 MOTOR 1 DRIVER LEFT, J302 MOTOR 2 DRIVER LEFT, J303 MOTOR 1 DRIVER RIGHT, J304 MOTOR 2 DRIVER RIGHT

Commit message: final schematic and layout
Parts:
- J301, J302, J303, J304: footprint (none) -> skittle_pnp:RHDR8W80P0X254_1X8_2082X254X850P
Connections:
- net GND: now also J303.1 (Pin_1)
Changed lines of the file:
@@
 F 0 "J301" H 3050 2450 50  0000 L CNN
 F 1 "MOTOR 1 DRIVER LEFT" V 3200 1500 50  0000 L CNN
-F 2 "" H 3100 2050 50  0001 C CNN
+F 2 "skittle_pnp:RHDR8W80P0X254_1X8_2082X254X850P" H 3100 2050 50  0001 C CNN
 F 3 "~" H 3100 2050 50  0001 C CNN
 	1    3100 2050
@@
 F 0 "J302" H 3050 4150 50  0000 L CNN
 F 1 "MOTOR 2 DRIVER LEFT" V 3200 3200 50  0000 L CNN
-F 2 "" H 3100 3750 50  0001 C CNN
+F 2 "skittle_pnp:RHDR8W80P0X254_1X8_2082X254X850P" H 3100 3750 50  0001 C CNN
 F 3 "~" H 3100 3750 50  0001 C CNN
 	1    3100 3750
 	1    0    0    -1
-$EndComp
-$Comp
-L Connector_Generic:Conn_01x08 J?
-U 1 1 61FEBEC9
-P 4000 2150
-AR Path="/619053FC/61FEBEC9" Ref="J?"  Part="1"
-AR Path="/61FBB307/61FEBEC9" Ref="J303"  Part="1"
-F 0 "J303" H 4000 1650 50  0000 C CNN
-F 1 "MOTOR 1 DRIVER RIGHT" V 4100 2150 50  0000 C CNN
-F 2 "" H 4000 2150 50  0001 C CNN
-F 3 "~" H 4000 2150 50  0001 C CNN
-	1    4000 2150
-	-1   0    0    1
 $EndComp
 $Comp
@@
 F 0 "J304" H 4000 3350 50  0000 C CNN
 F 1 "MOTOR 2 DRIVER RIGHT" V 4100 3850 50  0000 C CNN
-F 2 "" H 4000 3850 50  0001 C CNN
+F 2 "skittle_pnp:RHDR8W80P0X254_1X8_2082X254X850P" H 4000 3850 50  0001 C CNN
 F 3 "~" H 4000 3850 50  0001 C CNN
 	1    4000 3850
@@
 Text Notes 5300 3050 2    50   ~ 0
 logic power supply
-Text Notes 5450 2950 0    50   ~ 0
+Text Notes 10300 3150 0    50   ~ 0
 motor power supply
 Text Notes 1200 1450 0    50   ~ 0
 do we need pullup resistors on the enable pins to disable the internal fet outputs?
+$Comp
+L Connector_Generic:Conn_01x08 J?
+U 1 1 61FEBEC9
+P 4000 2150
+AR Path="/619053FC/61FEBEC9" Ref="J?"  Part="1"
+AR Path="/61FBB307/61FEBEC9" Ref="J303"  Part="1"
+F 0 "J303" H 4000 1650 50  0000 C CNN
+F 1 "MOTOR 1 DRIVER RIGHT" V 4100 2150 50  0000 C CNN
+F 2 "skittle_pnp:RHDR8W80P0X254_1X8_2082X254X850P" H 4000 2150 50  0001 C CNN
+F 3 "~" H 4000 2150 50  0001 C CNN
+	1    4000 2150
+	-1   0    0    1
+$EndComp
+$Comp
+L power:GND #PWR?
+U 1 1 61AD12EC
+P 4350 2550
+F 0 "#PWR?" H 4350 2300 50  0001 C CNN
+F 1 "GND" H 4355 2377 50  0000 C CNN
+F 2 "" H 4350 2550 50  0001 C CNN
+F 3 "" H 4350 2550 50  0001 C CNN
+	1    4350 2550
+	1    0    0    -1
+$EndComp
+Wire Wire Line
+	4200 2450 4350 2450
+Wire Wire Line
+	4350 2450 4350 2550
 $EndSCHEMATC
