File: hardware/main_board/_autosave-main_board.kicad_pcb (KiCad board)
At the start: 2 copper layers, 119.4 x 110.7 mm, 53 parts, among them J301 MOTOR 1 DRIVER LEFT, J302 MOTOR 2 DRIVER LEFT, J303 MOTOR 1 DRIVER RIGHT, J304 MOTOR 2 DRIVER RIGHT, J401 Conn_01x20, J402 Conn_01x20, J403 I2C, J404 USART 1, J405 USART 2, J406 SERVO, J407 MOTOR 1, J408 POWER, J409 SKITTLE PICKUP, J410 MOTOR 2, J412 LIMIT SWITCHES, Q501 SSM3K333R, U201 LM1117-5.0, U202 LM1117-3.3

Commit message: added final schematic and layout
Connections:
- J401 pad 18: +5V -> Net-(J401-Pad18)
Changed lines of the file:
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@@
     (zones 0)
     (modules 53)
-    (nets 56)
+    (nets 57)
   )
   (page A4)
@@
   (net 54 "/Motor Drivers/MOTOR1_~RESET")
   (net 55 "/Motor Drivers/MOTOR2_~RESET")
+  (net 56 "Net-(J401-Pad18)")
   (net_class Default "This is the default net class."
     (clearance 0.2)
@@
     (add_net MOTOR2_~EN)
     (add_net "Net-(F401-Pad1)")
+    (add_net "Net-(J401-Pad18)")
     (add_net "Net-(J406-Pad1)")
     (add_net "Net-(R201-Pad2)")
@@
       (net 10 /STM32_and_Connectors/PB9))
     (pad 18 thru_hole circle (at 43.18 0 270) (size 2.025 2.025) (drill 1.35) (layers *.Cu *.Mask)
-      (net 3 +5V))
+      (net 56 "Net-(J401-Pad18)"))
     (pad 19 thru_hole circle (at 45.72 0 270) (size 2.025 2.025) (drill 1.35) (layers *.Cu *.Mask)
       (net 2 GND))
